Commit message: add new files for creating logsitics_warehouse map and modify files for multi robot nav2 stack

File: src/virtual_lab/urdf/mogi_bot_single.urdf.xacro (robot description, xacro)
@@ -2,9 +2,4 @@
 <robot name="mogi_bot" xmlns:xacro="http://www.ros.org/wiki/xacro">
   <!-- ========================================================= -->
-  <!-- ROBOT NAMESPACE -->
-  <!-- ========================================================= -->
-  <xacro:arg name="robot_name" default=""/>
-  <xacro:property name="robot_name" value="$(arg robot_name)"/>
-  <!-- ========================================================= -->
   <!-- GAZEBO + MATERIALS -->
   <!-- ========================================================= -->
@@ -14,14 +9,14 @@
   <!-- BASE FOOTPRINT -->
   <!-- ========================================================= -->
-  <link name="${robot_name}/base_footprint"/>
+  <link name="base_footprint"/>
   <!-- ========================================================= -->
   <!-- BASE LINK -->
   <!-- ========================================================= -->
-  <joint name="${robot_name}/base_footprint_joint" type="fixed">
+  <joint name="base_footprint_joint" type="fixed">
     <origin xyz="0 0 0" rpy="0 0 0"/>
-    <parent link="${robot_name}/base_footprint"/>
-    <child link="${robot_name}/base_link"/>
-  </joint>
-  <link name="${robot_name}/base_link">
+    <parent link="base_footprint"/>
+    <child link="base_link"/>
+  </joint>
+  <link name="base_link">
     <pose>0 0 0.1 0 0 0</pose>
     <inertial>
@@ -48,5 +43,4 @@
       </geometry>
     </visual>
-    <!-- Rear caster -->
     <collision name="rear_caster_collision">
       <origin xyz="-0.15 0 -0.05" rpy="0 0 0"/>
@@ -61,5 +55,4 @@
       </geometry>
     </visual>
-    <!-- Front caster -->
     <collision name="front_caster_collision">
       <origin xyz="0.15 0 -0.05" rpy="0 0 0"/>
@@ -78,15 +71,13 @@
   <!-- LEFT WHEEL -->
   <!-- ========================================================= -->
-  <joint
-    type="continuous"
-    name="${robot_name}/left_wheel_joint">
+  <joint type="continuous" name="left_wheel_joint">
     <origin xyz="0 0.15 0" rpy="0 0 0"/>
-    <child link="${robot_name}/left_wheel"/>
-    <parent link="${robot_name}/base_link"/>
+    <child link="left_wheel"/>
+    <parent link="base_link"/>
     <axis xyz="0 1 0"/>
     <limit effort="100" velocity="10"/>
     <dynamics damping="1.0" friction="1.0"/>
   </joint>
-  <link name="${robot_name}/left_wheel">
+  <link name="left_wheel">
     <inertial>
       <mass value="5.0"/>
@@ -116,15 +107,13 @@
   <!-- RIGHT WHEEL -->
   <!-- ========================================================= -->
-  <joint
-    type="continuous"
-    name="${robot_name}/right_wheel_joint">
+  <joint type="continuous" name="right_wheel_joint">
     <origin xyz="0 -0.15 0" rpy="0 0 0"/>
-    <child link="${robot_name}/right_wheel"/>
-    <parent link="${robot_name}/base_link"/>
+    <child link="right_wheel"/>
+    <parent link="base_link"/>
     <axis xyz="0 1 0"/>
     <limit effort="100" velocity="10"/>
     <dynamics damping="1.0" friction="1.0"/>
   </joint>
-  <link name="${robot_name}/right_wheel">
+  <link name="right_wheel">
     <inertial>
       <mass value="5.0"/>
@@ -154,5 +143,5 @@
   <!-- WHEEL FRICTION -->
   <!-- ========================================================= -->
-  <gazebo reference="${robot_name}/left_wheel">
+  <gazebo reference="left_wheel">
     <mu1>0.2</mu1>
     <mu2>0.2</mu2>
@@ -162,5 +151,5 @@
     <maxVel>1.0</maxVel>
   </gazebo>
-  <gazebo reference="${robot_name}/right_wheel">
+  <gazebo reference="right_wheel">
     <mu1>0.2</mu1>
     <mu2>0.2</mu2>
@@ -170,5 +159,5 @@
     <maxVel>1.0</maxVel>
   </gazebo>
-  <gazebo reference="${robot_name}/base_link">
+  <gazebo reference="base_link">
     <mu1>0.000002</mu1>
     <mu2>0.000002</mu2>
@@ -177,24 +166,20 @@
   <!-- IMU -->
   <!-- ========================================================= -->
-  <joint
-    name="${robot_name}/imu_joint"
-    type="fixed">
+  <joint name="imu_joint" type="fixed">
     <origin xyz="0 0 0" rpy="0 0 0"/>
-    <parent link="${robot_name}/base_link"/>
-    <child link="${robot_name}/imu_link"/>
-  </joint>
-  <link name="${robot_name}/imu_link"/>
+    <parent link="base_link"/>
+    <child link="imu_link"/>
+  </joint>
+  <link name="imu_link"/>
   <!-- ========================================================= -->
   <!-- LIDAR -->
   <!-- ========================================================= -->
-  <joint
-    type="fixed"
-    name="${robot_name}/scan_joint">
+  <joint type="fixed" name="scan_joint">
     <origin xyz="0 0 0.15" rpy="0 0 0"/>
-    <child link="${robot_name}/lidar_link"/>
-    <parent link="${robot_name}/base_link"/>
+    <child link="lidar_link"/>
+    <parent link="base_link"/>
     <axis xyz="0 1 0"/>
   </joint>
-  <link name="${robot_name}/lidar_link">
+  <link name="lidar_link">
     <inertial>
       <mass value="1e-5"/>
@@ -221,8 +206,5 @@
     </visual>
   </link>
-  <!-- ========================================================= -->
-  <!-- LIDAR GAZEBO SETTINGS -->
-  <!-- ========================================================= -->
-  <gazebo reference="${robot_name}/lidar_link">
+  <gazebo reference="lidar_link">
     <selfCollide>false</selfCollide>
     <mu1 value="0.05"/>
